File: kicad/orange_juice_board.kicad_sch (KiCad schematic)
At the start: 56 parts, among them J10 GPIO12_Head, J10 PWM_OUT1, J11 CONN_UART, J12 Conn_01x08, J12 PWM_OUT2, J13 GPIO6_Head, J14 GPIO11_Head, J15 PWM_OUT3, J2 DC_INPUT, J3 CONN_ADXL345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

Commit message: some progress
Parts:
- added J?: Zero 2 GPIO PINs 2, symbol Connector_Generic:Conn_01x03
Connections:
- net BUCK_OUT: now also J7.1 (Pin_1)
- net GND: now also J7.2 (Pin_2), J?.1 (Pin_1); no longer J7.12 (Pin_12)
- net GPIO12: now also J?.2 (Pin_2), J?.3 (Pin_3)
- net SPI1_CS: no longer J4.24 (Pin_24)
- net USB2_D+: now also J7.4 (Pin_4); no longer J7.10 (Pin_10)
- net USB2_D-: now also J7.3 (Pin_3); no longer J7.11 (Pin_11)
- net USB3_D+: now also J7.6 (Pin_6); no longer J7.8 (Pin_8)
- net USB3_D-: now also J7.5 (Pin_5); no longer J7.9 (Pin_9)
- new net SPI1_CS_1: J4.24 (Pin_24)
- no-connect marks 12 -> 4

Commit message: v0.8 bate version
Parts:
- removed J?: Zero 2 GPIO PINs 2, symbol Connector_Generic:Conn_01x03
- J10: value GPIO12_Head -> GPIO229_Head
- J13: value GPIO6_Head -> GPIO73_Head
- J14: value GPIO11_Head -> GPIO228_Head
Connections:
- net SPI1_CS_1 is gone; now on net SPI1_CS: J4.24 (Pin_24)
- net BUCK_OUT: no longer J7.1 (Pin_1)
- net GND: now also J7.12 (Pin_12); no longer J7.2 (Pin_2)
- net USB2_Conn_D+: now also USB1.7 (D+); no longer USB1.3 (D+)
- net USB2_Conn_D-: now also USB1.6 (D-); no longer USB1.2 (D-)
- net USB2_D+: now also J7.10 (Pin_10); no longer J7.4 (Pin_4)
- net USB2_D-: now also J7.11 (Pin_11); no longer J7.3 (Pin_3)
- net USB3_Conn_D+: now also USB1.3 (D+); no longer USB1.7 (D+)
- net USB3_Conn_D-: now also USB1.2 (D-); no longer USB1.6 (D-)
- net USB3_D+: now also J7.8 (Pin_8); no longer J7.6 (Pin_6)
- net USB3_D-: now also J7.9 (Pin_9); no longer J7.5 (Pin_5)
- net GPIO11 renamed GPIO228
- net GPIO12 renamed GPIO229
- net GPIO6 renamed GPIO73
- net GPIO_0_SDI renamed GPIO_69_SDI
- net GPIO_10 renamed GPIO_74
- net GPIO_18 renamed GPIO_78
- net GPIO_19 renamed GPIO_79
- net GPIO_1_CS renamed GPIO_70_CS
- net GPIO_2_CLK renamed GPIO_71_CLK
- net GPIO_3_SDO renamed GPIO_72_SDO
- no-connect marks 4 -> 12
Other:
- title: Orange Juice -> Orange Juice for Zero2
